Commit message: Adding all changes

File: dot_description/xacro/main.urdf.xacro (robot description, xacro)
@@ -401,5 +401,5 @@
         <origin rpy="0 0 0" xyz="0 0 0"/>
         <geometry>
-            <mesh filename="package://dot_description/mesh/tag0/tag0.dae" scale="0.45 0.45 1"/>
+            <mesh filename="package://dot_description/mesh/tag0/tag0.dae" scale="1 1 1"/>
         </geometry>
     </visual>
@@ -414,4 +414,5 @@
     <minDepth>0.001</minDepth>
 </gazebo>
+<!--
 <link name='platform_tag1'>
     <inertial>
@@ -438,5 +439,5 @@
     <maxVel>0.0</maxVel>
     <minDepth>0.001</minDepth>
-</gazebo>
+</gazebo> -->
 <link name='platform'>
     <inertial>
@@ -516,13 +517,13 @@
 </joint>
 <joint name='fixed_joint0' type='fixed'>
-    <origin rpy="0.0 0.0 0.0" xyz="-0.023 -0.023 0.008"/>
+    <origin rpy="0.0 0.0 0.0" xyz="0.00 0.00 0.008"/>
     <parent link="platform_mid"/>
     <child link="platform_tag0"/>
 </joint>
-<joint name='fixed_joint1' type='fixed'>
+<!-- <joint name='fixed_joint1' type='fixed'>
     <origin rpy="0.0 0.0 0.0" xyz="0.023 0.023 0.008"/>
     <parent link="platform_mid"/>
     <child link="platform_tag1"/>
-</joint>
+</joint> -->
 <transmission name="simple_trans1">
     <type>transmission_interface/SimpleTransmission</type>

File: dot_gazebo/urdf/cameras.urdf (robot description, URDF)
Before this commit: robot bot, 8 links, 7 joints
Links:
- added link april10, mass 0.002; visual mesh filename=package://dot_description/mesh/tag10/tag10.dae scale=1 1 1
- added link april11, mass 0.002; visual mesh filename=package://dot_description/mesh/tag11/tag11.dae scale=1 1 1
- added link april12, mass 0.002; visual mesh filename=package://dot_description/mesh/tag12/tag12.dae scale=1 1 1
- added link april13, mass 0.002; visual mesh filename=package://dot_description/mesh/tag13/tag13.dae scale=1 1 1
- added link april14, mass 0.002; visual mesh filename=package://dot_description/mesh/tag14/tag14.dae scale=1 1 1
- added link april15, mass 0.002; visual mesh filename=package://dot_description/mesh/tag15/tag15.dae scale=1 1 1
- added link april16, mass 0.002; visual mesh filename=package://dot_description/mesh/tag16/tag16.dae scale=1 1 1
- added link april17, mass 0.002; visual mesh filename=package://dot_description/mesh/tag17/tag17.dae scale=1 1 1
- added link april18, mass 0.002; visual mesh filename=package://dot_description/mesh/tag0/tag0.dae scale=1 1 1
- added link april19, mass 0.002; visual mesh filename=package://dot_description/mesh/tag1/tag1.dae scale=1 1 1
- added link april20, mass 0.002; visual mesh filename=package://dot_description/mesh/tag2/tag2.dae scale=1 1 1
- added link april21, mass 0.002; visual mesh filename=package://dot_description/mesh/tag3/tag3.dae scale=1 1 1
- added link april22, mass 0.002; visual mesh filename=package://dot_description/mesh/tag4/tag4.dae scale=1 1 1
- added link april23, mass 0.002; visual mesh filename=package://dot_description/mesh/tag5/tag5.dae scale=1 1 1
- added link april4, mass 0.002; visual mesh filename=package://dot_description/mesh/tag4/tag4.dae scale=1 1 1
- added link april5, mass 0.002; visual mesh filename=package://dot_description/mesh/tag5/tag5.dae scale=1 1 1
- added link april6, mass 0.002; visual mesh filename=package://dot_description/mesh/tag6/tag6.dae scale=1 1 1
- added link april7, mass 0.002; visual mesh filename=package://dot_description/mesh/tag7/tag7.dae scale=1 1 1
- added link april8, mass 0.002; visual mesh filename=package://dot_description/mesh/tag8/tag8.dae scale=1 1 1
- added link april9, mass 0.002; visual mesh filename=package://dot_description/mesh/tag9/tag9.dae scale=1 1 1
Joints:
- added joint apri10: type fixed, parent world, child april10, origin xyz=0.6096 -0.3048 0.04 rpy=0 0 0
- added joint apri11: type fixed, parent world, child april11, origin xyz=0.3048 0.3048 0.04 rpy=0 0 0
- added joint apri12: type fixed, parent world, child april12, origin xyz=0.6096 0.3048 0.04 rpy=0 0 0
- added joint apri13: type fixed, parent world, child april13, origin xyz=-0.9144 0 0.04 rpy=0 0 0
- added joint apri14: type fixed, parent world, child april14, origin xyz=-0.9144 0.6096 0.04 rpy=0 0 0
- added joint apri15: type fixed, parent world, child april15, origin xyz=-0.9144 -0.6096 0.04 rpy=0 0 0
- added joint apri16: type fixed, parent world, child april16, origin xyz=0.9144 0.3048 0.04 rpy=0 0 0
- added joint apri17: type fixed, parent world, child april17, origin xyz=0.9144 -0.3048 0.04 rpy=0 0 0
- added joint apri18: type fixed, parent world, child april18, origin xyz=0.3048 0.6096 0.04 rpy=0 0 0
- added joint apri19: type fixed, parent world, child april19, origin xyz=-0.3048 0.6096 0.04 rpy=0 0 0
- added joint apri20: type fixed, parent world, child april20, origin xyz=-0.3048 0 0.04 rpy=0 0 0
- added joint apri21: type fixed, parent world, child april21, origin xyz=0.3048 0 0.04 rpy=0 0 0
- added joint apri22: type fixed, parent world, child april22, origin xyz=-0.3048 -0.6096 0.04 rpy=0 0 0
- added joint apri23: type fixed, parent world, child april23, origin xyz=0.3048 -0.6096 0.04 rpy=0 0 0
- added joint apri4: type fixed, parent world, child april4, origin xyz=0 0.3048 0.04 rpy=0 0 0
- added joint apri5: type fixed, parent world, child april5, origin xyz=-0.9144 -0.3048 0.04 rpy=0 0 0
- added joint apri6: type fixed, parent world, child april6, origin xyz=-0.6096 -0.3048 0.04 rpy=0 0 0
- added joint apri7: type fixed, parent world, child april7, origin xyz=-0.3048 -0.3048 0.04 rpy=0 0 0
- added joint apri8: type fixed, parent world, child april8, origin xyz=0 -0.3048 0.04 rpy=0 0 0
- added joint apri9: type fixed, parent world, child april9, origin xyz=0.3048 -0.3048 0.04 rpy=0 0 0
- joint apri1: origin xyz=0 0 0.04 rpy=0 0 0 -> xyz=-0.9144 0.3048 0.04 rpy=0 0 0
- joint apri2: origin xyz=0.6096 0 0.04 rpy=0 0 0 -> xyz=-0.6096 0.3048 0.04 rpy=0 0 0
- joint apri3: origin xyz=-0.6096 0 0.04 rpy=0 0 0 -> xyz=-0.3048 0.3048 0.04 rpy=0 0 0
